Commit message: add robot FK example for irb4600 with track and GoFa

File: robots/abb_irb4600_40_255_with_linear_track/urdf/abb_irb4600_40_255_with_linear_track.urdf (robot description, URDF)
Before this commit: robot ECL_robot1_with_track, 14 links, 13 joints
Links:
- link linear_axis_base_link: geometry collision mesh filename=package://abb_irb4600_40_255_with_linear_track/meshes/colli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; visual mesh filename=package://abb_irb4600_40_255_with_linear_track/meshes/visua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
- link linear_axis_carriage: geometry collision mesh filename=package://abb_irb4600_40_255_with_linear_track/meshes/colli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; visual mesh filename=package://abb_irb4600_40_255_with_linear_track/meshes/visua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
